Commit message: imu and dynamic config are ok

File: src/bicycle_urdf/urdf/bicycle_urdf.urdf (robot description, URDF)
Before this commit: robot bicycle_urdf, 7 links, 6 joints
Links:
- link base_link: mass 9.99999999988803E-11 -> None
- link j1: mass 3.74892369130333 -> 3.6404
- link j2: mass 0.640712092512939 -> 0.68174
- link j3: mass 1.42289136054877 -> 1.4336
- link j4: mass 1.46485195200999 -> 1.4778
- link j5: mass 0.0388487185787584 -> 0.037231
- link j6: mass 0.0447533363490518 -> 0.044753
Joints:
- joint j1: axis 0 0 0 -> 1 0 0; limit (none) -> lower=-1.57 upper=1.57 effort=0 velocity=0; origin xyz=0 0 0.57631 rpy=-1.3451 1.5708 -1.3451 -> xyz=0 0 0 rpy=0 0 0; type fixed -> revolute
- joint j2: origin xyz=-0.31644 0 0.35759 rpy=3.1416 -1.2334 -3.1416 -> xyz=0.38509 0.000175 0.89724 rpy=0 -0.312 0
- joint j3: axis 0 0 1 -> 0 1 0; origin xyz=0.00011884 -0.001 -0.5832 rpy=-1.5708 0.36721 0 -> xyz=0.00011884 -0.001 -0.5832 rpy=0 0.312 0
- joint j4: axis 0 0 -1 -> 0 -1 0; origin xyz=0.25864 -0.000175 -0.43731 rpy=-1.5708 -1.5409 0 -> xyz=-0.42413 0 0.3425 rpy=0 0 0
- joint j5: origin xyz=-0.26811 0 0.4581 rpy=3.1416 -1.5143 3.1416 -> xyz=0.48435 0.00017515 0.84618 rpy=0 0 0
- joint j6: origin xyz=0.081171 -0.00088133 0.016378 rpy=3.1416 1.3963 3.1416 -> xyz=0.068861 -0.00088133 0.018549 rpy=0 0.17453 0
